File: Main_light_system/Eagle/Main_PCB.sch (EAGLE design)
At the start: 14 parts, among them U1 TPS54308DDCT, U2 TPS54308DDCT

Commit message: update main pcb
Parts:
- added U$1: BERRY_PI_ZERO_W, Main_lib:BERRY_PI_ZERO_W
- added U$2: ToSensors, Main_lib:MODULARCONNECTOR
- added U$3: ToLampDrivers, Main_lib:MODULARCONNECTOR
- added U$4, U$5: PARALLELHEADER, Main_lib:PARALLELHEADER
Connections:
- removed net +5V: COUT1.+, L1.2, RFBT1.2
- new net 3.3V: U$1.3V3@1, U$1.3V3@2, U$2.1, U$3.1, U$4.12, U$4.20
- new net 5V: COUT1.+, L1.2, RFBT1.2, U$1.5V@1, U$1.5V@2, U$5.1, U$5.2
- new net N$10: U$1.GPIO13, U$4.4
- new net N$11: U$1.GPIO6, U$4.5
- new net N$12: U$1.GPIO5, U$4.6
- new net N$13: U$1.ID_SD, U$4.7
- new net N$15: U$1.GPIO11, U$4.9
- new net N$16: U$1.GPIO9, U$4.10
- new net N$17: U$1.GPIO10, U$4.11
- new net N$19: U$1.GPIO22, U$4.13
- new net N$20: U$1.GPIO27, U$4.14
- new net N$21: U$1.GPIO17, U$4.15
- new net N$23: U$1.GPIO4, U$4.17
- new net N$26: U$1.GPIO14, U$5.4
- new net N$27: U$1.GPIO15, U$5.5
- new net N$28: U$1.GPIO18, U$5.6
- new net N$30: U$1.GPIO23, U$5.8
- new net N$31: U$1.GPIO24, U$5.9
- new net N$33: U$1.GPIO25, U$5.11
- new net N$34: U$1.GPIO8, U$5.12
- new net N$35: U$1.GPIO7, U$5.13
- new net N$36: U$1.ID_SC, U$5.14
- new net N$38: U$1.GPIO12, U$5.16
- new net N$40: U$1.GPIO16, U$5.18
- new net N$41: U$1.GPIO20, U$5.19
- new net N$42: U$1.GPIO21, U$5.20
- new net N$8: U$1.GPIO26, U$4.2
- new net N$9: U$1.GPIO19, U$4.3
- new net SCL: U$1.GPIO3, U$2.3, U$3.3, U$4.18
- new net SDA: U$1.GPIO2, U$2.2, U$3.2, U$4.19
- net GND: now also U$1.GND@1, U$1.GND@2, U$1.GND@3, U$1.GND@4, U$1.GND@5, U$1.GND@6, U$1.GND@7, U$1.GND@8, U$2.8, U$3.8, U$4.1, U$4.16, U$4.8, U$5.10, U$5.15, U$5.17, U$5.3, U$5.7

Commit message: main pcb update
Connections:
- net 3.3V: now also U$2.8; no longer U$3.1
- net 5V: now also U$3.1, U$3.8
- net GND: now also U$2.2, U$2.7, U$3.2, U$3.7; no longer U$2.8, U$3.8
- net SCL: now also U$2.4, U$2.5, U$3.4, U$3.5; no longer U$2.3, U$3.3
- net SDA: now also U$2.3, U$2.6, U$3.3, U$3.6; no longer U$2.2, U$3.2
Other:
- moved on the sheet: U$2, U$3
