File: Main_light_system/Eagle/Main_PCB.sch (EAGLE design)
At the start: 19 parts, among them U1 TPS54308DDCT, U2 TPS54308DDCT

Commit message: schema main update
Parts:
- added J1: PUSH_TERMINAL_2WAYS, Main_lib:PUSH_TERMINAL_2WAYS
- U$2: value ToSensors -> LinkerVrouwtje
- U$3: value ToLampDrivers -> RechterMannetje
Connections:
- net +12V: now also J1.1
- net 3.3V: now also U$2.3, U$2.4, U$3.3, U$3.4; no longer U$2.1, U$2.8
- net 5V: now also U$2.1, U$2.2, U$3.2; no longer U$3.8
- net GND: now also J1.2, U$2.8, U$3.8; no longer U$2.2, U$3.2
- net SCL: now also U$2.6, U$3.6; no longer U$2.4, U$2.5, U$3.4, U$3.5
- net SDA: now also U$2.5, U$3.5; no longer U$2.3, U$2.6, U$3.3, U$3.6
Other:
- moved on the sheet: U$2, U$3

Commit message: PCB Main bijna af
Connections:
- removed net +3V3: COUT2.+, L2.2, RFBT2.2
- new net 5V@2: U$1.5V@2, U$5.2
- new net N$14: U$1.3V3@2, U$4.12
- new net N$7: U$1.3V3@1, U$4.20
- net 3.3V: now also COUT2.+, L2.2, RFBT2.2; no longer U$1.3V3@1, U$1.3V3@2, U$4.12, U$4.20
- net 5V: no longer U$1.5V@2, U$5.2
Changed lines of the file:
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@@
 <part name="CBST2" library="Main_lib" deviceset="C-0603" device="" value="100nF"/>
 <part name="GND1" library="supply1" library_urn="urn:adsk.eagle:library:371" deviceset="GND" device=""/>
-<part name="+3V1" library="supply1" library_urn="urn:adsk.eagle:library:371" deviceset="+3V3" device=""/>
+<part name="+3V1" library="supply1" library_urn="urn:adsk.eagle:library:371" deviceset="+3V3" device="" value="3.3V"/>
 <part name="P+1" library="supply1" library_urn="urn:adsk.eagle:library:371" deviceset="+12V" device=""/>
 <part name="GND2" library="supply1" library_urn="urn:adsk.eagle:library:371" deviceset="GND" device=""/>
@@
 <part name="U$2" library="Main_lib" deviceset="MODULARCONNECTOR" device="" value="LinkerVrouwtje"/>
 <part name="U$3" library="Main_lib" deviceset="MODULARCONNECTOR" device="" value="RechterMannetje"/>
-<part name="SUPPLY1" library="SparkFun-PowerSymbols" library_urn="urn:adsk.eagle:library:530" deviceset="3.3V" device=""/>
 <part name="SUPPLY2" library="SparkFun-PowerSymbols" library_urn="urn:adsk.eagle:library:530" deviceset="5V" device=""/>
 <part name="GND9" library="SparkFun-PowerSymbols" library_urn="urn:adsk.eagle:library:530" deviceset="GND" device=""/>
@@
 <attribute name="NAME" x="10.16" y="80.01" size="1.778" layer="95"/>
 <attribute name="VALUE" x="10.16" y="53.34" size="1.778" layer="96"/>
-</instance>
-<instance part="SUPPLY1" gate="G$1" x="71.12" y="83.82" smashed="yes">
-<attribute name="VALUE" x="71.12" y="86.614" size="1.778" layer="96" align="bottom-center"/>
 </instance>
 <instance part="SUPPLY2" gate="G$1" x="106.68" y="88.9" smashed="yes">
@@
 <net name="3.3V" class="0">
 <segment>
-<pinref part="U$1" gate="G$1" pin="3V3@1"/>
-<pinref part="U$4" gate="G$1" pin="20"/>
-<wire x1="55.88" y1="76.2" x2="71.12" y2="76.2" width="0.1524" layer="91"/>
-<pinref part="U$1" gate="G$1" pin="3V3@2"/>
-<pinref part="U$4" gate="G$1" pin="12"/>
-<wire x1="71.12" y1="76.2" x2="73.66" y2="76.2" width="0.1524" layer="91"/>
-<wire x1="55.88" y1="55.88" x2="71.12" y2="55.88" width="0.1524" layer="91"/>
-<wire x1="71.12" y1="55.88" x2="73.66" y2="55.88" width="0.1524" layer="91"/>
-<wire x1="71.12" y1="76.2" x2="71.12" y2="55.88" width="0.1524" layer="91"/>
-<junction x="71.12" y="76.2"/>
-<junction x="71.12" y="55.88"/>
-<pinref part="SUPPLY1" gate="G$1" pin="3.3V"/>
-<wire x1="71.12" y1="83.82" x2="71.12" y2="76.2" width="0.1524" layer="91"/>
-</segment>
-<segment>
 <pinref part="U$3" gate="G$1" pin="3"/>
 <pinref part="U$2" gate="G$1" pin="3"/>
@@
 <wire x1="106.68" y1="88.9" x2="106.68" y2="76.2" width="0.1524" layer="91"/>
 <junction x="106.68" y="76.2"/>
-<pinref part="U$1" gate="G$1" pin="5V@2"/>
-<pinref part="U$5" gate="G$1" pin="2"/>
-<wire x1="121.92" y1="73.66" x2="106.68" y2="73.66" width="0.1524" layer="91"/>
-<wire x1="106.68" y1="73.66" x2="104.14" y2="73.66" width="0.1524" layer="91"/>
-<wire x1="106.68" y1="76.2" x2="106.68" y2="73.66" width="0.1524" layer="91"/>
-<junction x="106.68" y="73.66"/>
 </segment>
 <segment>
@@
 </segment>
 </net>
+<net name="N$7" class="0">
+<segment>
+<pinref part="U$1" gate="G$1" pin="3V3@1"/>
+<pinref part="U$4" gate="G$1" pin="20"/>
+<wire x1="55.88" y1="76.2" x2="73.66" y2="76.2" width="0.1524" layer="91"/>
+</segment>
+</net>
+<net name="N$14" class="0">
+<segment>
+<pinref part="U$1" gate="G$1" pin="3V3@2"/>
+<pinref part="U$4" gate="G$1" pin="12"/>
+<wire x1="55.88" y1="55.88" x2="73.66" y2="55.88" width="0.1524" layer="91"/>
+</segment>
+</net>
+<net name="5V@2" class="0">
+<segment>
+<pinref part="U$1" gate="G$1" pin="5V@2"/>
+<pinref part="U$5" gate="G$1" pin="2"/>
+<wire x1="121.92" y1="73.66" x2="104.14" y2="73.66" width="0.1524" layer="91"/>
+</segment>
+</net>
 </nets>
 </sheet>
@@
 </segment>
 </net>
-<net name="+3V3" class="0">
+<net name="3.3V" class="0">
 <segment>
 <pinref part="L2" gate="G$1" pin="2"/>
@@
 <wire x1="127" y1="43.18" x2="142.24" y2="43.18" width="0.1524" layer="91"/>
 <junction x="127" y="43.18"/>
-</segment>
-</net>
+<label x="119.38" y="45.72" size="1.778" layer="95"/>
+</segment>
+</net>

Commit message: pcb main af?
Parts:
- J1: value PUSH_TERMINAL_2WAYS -> Vin
- U$2: value LinkerVrouwtje -> Female
- U$3: value RechterMannetje -> MALE
- U$4: value PARALLELHEADER -> ODD PINS
- U$5: value PARALLELHEADER -> EVEN PINS
Changed lines of the file:
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@@
 <drawing>
 <settings>
-<setting alwaysvectorfont="yes"/>
+<setting alwaysvectorfont="no"/>
 <setting verticaltext="up"/>
 </settings>
@@
 <part name="CBST2" library="Main_lib" deviceset="C-0603" device="" value="100nF"/>
 <part name="GND1" library="supply1" library_urn="urn:adsk.eagle:library:371" deviceset="GND" device=""/>
-<part name="+3V1" library="supply1" library_urn="urn:adsk.eagle:library:371" deviceset="+3V3" device="" value="3.3V"/>
+<part name="3.3V1" library="supply1" library_urn="urn:adsk.eagle:library:371" deviceset="+3V3" device="" value="3.3V"/>
 <part name="P+1" library="supply1" library_urn="urn:adsk.eagle:library:371" deviceset="+12V" device=""/>
 <part name="GND2" library="supply1" library_urn="urn:adsk.eagle:library:371" deviceset="GND" device=""/>
@@
 <part name="GND8" library="supply1" library_urn="urn:adsk.eagle:library:371" deviceset="GND" device=""/>
 <part name="U$1" library="Main_lib" deviceset="BERRY_PI_ZERO_W" device=""/>
-<part name="U$2" library="Main_lib" deviceset="MODULARCONNECTOR" device="" value="LinkerVrouwtje"/>
-<part name="U$3" library="Main_lib" deviceset="MODULARCONNECTOR" device="" value="RechterMannetje"/>
+<part name="U$2" library="Main_lib" deviceset="MODULARCONNECTOR" device="" value="Female"/>
+<part name="U$3" library="Main_lib" deviceset="MODULARCONNECTOR" device="" value="MALE"/>
 <part name="SUPPLY2" library="SparkFun-PowerSymbols" library_urn="urn:adsk.eagle:library:530" deviceset="5V" device=""/>
 <part name="GND9" library="SparkFun-PowerSymbols" library_urn="urn:adsk.eagle:library:530" deviceset="GND" device=""/>
 <part name="GND10" library="SparkFun-PowerSymbols" library_urn="urn:adsk.eagle:library:530" deviceset="GND" device=""/>
-<part name="U$4" library="Main_lib" deviceset="PARALLELHEADER" device=""/>
-<part name="U$5" library="Main_lib" deviceset="PARALLELHEADER" device=""/>
+<part name="U$4" library="Main_lib" deviceset="PARALLELHEADER" device="" value="ODD PINS"/>
+<part name="U$5" library="Main_lib" deviceset="PARALLELHEADER" device="" value="EVEN PINS"/>
 <part name="SUPPLY3" library="SparkFun-PowerSymbols" library_urn="urn:adsk.eagle:library:530" deviceset="3.3V" device=""/>
 <part name="GND12" library="SparkFun-PowerSymbols" library_urn="urn:adsk.eagle:library:530" deviceset="GND" device=""/>
@@
 <part name="U$8" library="Main_lib" deviceset="SCL" device=""/>
 <part name="SUPPLY8" library="SparkFun-PowerSymbols" library_urn="urn:adsk.eagle:library:530" deviceset="5V" device=""/>
-<part name="J1" library="Main_lib" deviceset="PUSH_TERMINAL_2WAYS" device=""/>
+<part name="J1" library="Main_lib" deviceset="PUSH_TERMINAL_2WAYS" device="" value="Vin"/>
 <part name="GND13" library="SparkFun-PowerSymbols" library_urn="urn:adsk.eagle:library:530" deviceset="GND" device=""/>
 <part name="P+3" library="supply1" library_urn="urn:adsk.eagle:library:371" deviceset="+12V" device=""/>
@@
 <attribute name="VALUE" x="106.68" y="7.62" size="1.778" layer="96"/>
 </instance>
-<instance part="+3V1" gate="G$1" x="144.78" y="43.18" smashed="yes" rot="R270">
+<instance part="3.3V1" gate="G$1" x="144.78" y="43.18" smashed="yes" rot="R270">
 <attribute name="VALUE" x="139.7" y="45.72" size="1.778" layer="96"/>
 </instance>
@@
 <pinref part="COUT2" gate="A" pin="+"/>
 <wire x1="127" y1="43.18" x2="127" y2="35.56" width="0.1524" layer="91"/>
-<pinref part="+3V1" gate="G$1" pin="+3V3"/>
+<pinref part="3.3V1" gate="G$1" pin="+3V3"/>
 <wire x1="127" y1="43.18" x2="142.24" y2="43.18" width="0.1524" layer="91"/>
 <junction x="127" y="43.18"/>
@@
 </sheet>
 </sheets>
+<errors>
+</errors>
 </schematic>
 </drawing>

Commit message: gerbers
Parts:
- U$4: value ODD PINS -> ODD
- U$5: value EVEN PINS -> EVEN
Changed lines of the file:
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@@
 <drawing>
 <settings>
-<setting alwaysvectorfont="no"/>
+<setting alwaysvectorfont="yes"/>
 <setting verticaltext="up"/>
 </settings>
@@
 <part name="GND9" library="SparkFun-PowerSymbols" library_urn="urn:adsk.eagle:library:530" deviceset="GND" device=""/>
 <part name="GND10" library="SparkFun-PowerSymbols" library_urn="urn:adsk.eagle:library:530" deviceset="GND" device=""/>
-<part name="U$4" library="Main_lib" deviceset="PARALLELHEADER" device="" value="ODD PINS"/>
-<part name="U$5" library="Main_lib" deviceset="PARALLELHEADER" device="" value="EVEN PINS"/>
+<part name="U$4" library="Main_lib" deviceset="PARALLELHEADER" device="" value="ODD"/>
+<part name="U$5" library="Main_lib" deviceset="PARALLELHEADER" device="" value="EVEN"/>
 <part name="SUPPLY3" library="SparkFun-PowerSymbols" library_urn="urn:adsk.eagle:library:530" deviceset="3.3V" device=""/>
 <part name="GND12" library="SparkFun-PowerSymbols" library_urn="urn:adsk.eagle:library:530" deviceset="GND" device=""/>
