File: Main_light_system/Eagle/Main_PCB.brd (EAGLE design)
At the start: 160 x 100 mm, 20 parts, among them J1 PUSH_TERMINAL_2WAYS, U1 TPS54308DDCT, U2 TPS54308DDCT

Commit message: PCB Main bijna af
Parts:
- moved U$3 131.4 mm to (100.9, 25.0), flipped to the bottom, turned to 90 degrees
- moved U$1 110.2 mm to (64.0, 37.5)
- moved U$4 110.2 mm to (63.8, 47.5), turned to 180 degrees
- moved U$5 106.0 mm to (64.0, 43.9)
- moved CIN1 105.1 mm to (23.9, 4.53), turned to 90 degrees
- moved RFBT1 100.6 mm to (11.9, 10.4), turned to 90 degrees
- moved CBST1 97.8 mm to (16.7, 8.16)
- moved J1 96.7 mm to (41.0, 4.45), turned to 270 degrees
- moved COUT2 90.3 mm to (23.8, 33.2), turned to 180 degrees
- moved RFBB1 87.0 mm to (12.4, 4.66)
- moved CBST2 85.4 mm to (15.2, 40.5), turned to 180 degrees
- moved U1 80.3 mm to (16.9, 4.66), turned to 90 degrees
- moved RFBB2 77.3 mm to (22.6, 42.6), turned to 180 degrees
- moved COUT1 75.6 mm to (9.85, 15.8)
- moved U$2 56.3 mm to (3.10, 25.0), turned to 90 degrees
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Connections:
- removed net +3V3: COUT2.+, L2.2, RFBT2.2
- new net 5V@2: U$1.4, U$5.2
- new net N$14: U$1.17, U$4.12
- new net N$7: U$1.1, U$4.20
- net 3.3V: now also COUT2.+, L2.2, RFBT2.2; no longer U$1.1, U$1.17, U$4.12, U$4.20
- net 5V: no longer U$1.4, U$5.2
Routing:
- net 5V: track 0.00 -> 196.3 mm
- net SCL: track 0.00 -> 185.4 mm
- net SDA: track 0.00 -> 168.8 mm
- net 3.3V: track 0.00 -> 125.8 mm
- net +12V: track 0.00 -> 76.9 mm
- net GND: track 0.00 -> 17.3 mm
- net N$6: track 0.00 -> 13.8 mm
- net N$4: track 0.00 -> 13.7 mm
- net N$9: track 0.00 -> 12.1 mm
- net N$16: track 0.00 -> 12.1 mm
- net N$21: track 0.00 -> 12.1 mm
- net N$20: track 0.00 -> 12.1 mm
- net N$19: track 0.00 -> 12.1 mm
- net N$14: track 0.00 -> 12.1 mm
- net N$13: track 0.00 -> 12.1 mm
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- added copper zone on layer 1, net GND
- added copper zone on layer 16, net GND
Other:
- board size 160 x 100 mm -> 107 x 50 mm

Commit message: pcb main af?
Parts:
- J1: value PUSH_TERMINAL_2WAYS -> Vin
- U$2: value LinkerVrouwtje -> Female
- U$3: value RechterMannetje -> MALE
- U$4: value PARALLELHEADER -> ODD PINS
- U$5: value PARALLELHEADER -> EVEN PINS
- moved RFBB1 21.2 mm to (29.1, 17.7)
- moved RFBT1 21.1 mm to (29.9, 21.4)
- moved COUT2 13.4 mm to (17.8, 45.2)
- moved CIN2 12.8 mm to (18.6, 35.9), turned to 270 degrees
- moved U2 12.8 mm to (25.1, 36.1), turned to 0 degrees
- moved CBST2 11.0 mm to (26.2, 39.5)
- moved RFBT2 10.8 mm to (29.1, 46.2), turned to 90 degrees
- moved CBST1 10.8 mm to (26.7, 12.2), turned to 180 degrees
- moved U1 8.94 mm to (24.9, 8.66), turned to 0 degrees
- moved L1 8.25 mm to (10.9, 13.1)
- moved COUT1 7.81 mm to (14.8, 21.8), turned to 180 degrees
- moved CIN1 6.40 mm to (18.9, 8.53), turned to 270 degrees
- moved RFBB2 6.01 mm to (28.6, 43.0), turned to 0 degrees
- moved J1 6.00 mm to (47.0, 4.45)
- moved L2 5.66 mm to (10.5, 36.9), turned to 270 degrees
Routing:
- net +12V: track 76.9 -> 0.00 mm
- net 3.3V: track 125.8 -> 141.9 mm
- net N$3: track 10.3 -> 0.00 mm, vias 0 -> 8
- net N$1: track 9.82 -> 0.00 mm, vias 0 -> 10
- net GND: track 17.3 -> 12.1 mm, vias 0 -> 12
- net 5V: track 196.3 -> 192.3 mm
- net SCL: track 185.4 -> 189.2 mm
- net N$4: track 13.7 -> 11.6 mm
- net N$6: track 13.8 -> 15.2 mm
- net N$5: track 2.30 -> 3.16 mm
- added copper zone on layer 1, net +12V
- added copper zone on layer 1, net 3.3V
- added copper zone on layer 1, net 5V
- added copper zone on layer 1, net N$1
- added copper zone on layer 16, net N$1
- added copper zone on layer 1, net N$3
- added copper zone on layer 16, net N$3
Other:
- board size 107 x 50 mm -> 104 x 50 mm
- board text added: "Basile Berckmoes"
- board text added: "Frederik Callens"
- board text added: "KULeuven 2019"
- board text added: "Main PCB"

Commit message: gerbers
Parts:
- U$4: value ODD PINS -> ODD
- U$5: value EVEN PINS -> EVEN
