File: Sensor_light_system/Eagle/schema Light_system.brd (EAGLE design)
At the start: 60 x 50 mm, 23 parts, among them IC1 STM32F030C8T6TR, J1 12_WAY_CON

Commit message: eagel
Routing:
- net +3V3: track 160.2 -> 162.8 mm, vias 3 -> 4
Changed lines of the file:
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@@
 <wire x1="43.18" y1="23.114" x2="30.48" y2="23.114" width="1.27" layer="16"/>
 <wire x1="30.48" y1="23.114" x2="22.86" y2="23.114" width="1.27" layer="16"/>
-<wire x1="22.86" y1="23.114" x2="4.986" y2="23.114" width="1.27" layer="16"/>
+<wire x1="22.86" y1="23.114" x2="8.89" y2="23.114" width="1.27" layer="16"/>
+<wire x1="8.89" y1="23.114" x2="4.986" y2="23.114" width="1.27" layer="16"/>
 <wire x1="4.986" y1="23.114" x2="4.37" y2="23.73" width="1.27" layer="16"/>
 <wire x1="4.37" y1="23.73" x2="1.83" y2="23.73" width="1.27" layer="16"/>
 <wire x1="20.32" y1="45.72" x2="20.32" y2="43.18" width="1.016" layer="1"/>
 <wire x1="12.7" y1="6.35" x2="11.43" y2="7.62" width="0.3048" layer="1"/>
-<wire x1="11.43" y1="7.62" x2="11.43" y2="25.4" width="0.3048" layer="1"/>
+<wire x1="11.43" y1="7.62" x2="11.43" y2="22.86" width="0.3048" layer="1"/>
+<wire x1="11.43" y1="22.86" x2="11.43" y2="25.4" width="0.3048" layer="1"/>
 <wire x1="21.38" y1="29.638" x2="21.38" y2="30.56" width="0.3048" layer="1"/>
 <wire x1="21.38" y1="30.56" x2="18.985" y2="32.955" width="0.3048" layer="1"/>
@@
 <wire x1="18.985" y1="38.035" x2="18.985" y2="32.955" width="1.016" layer="1"/>
 <wire x1="20.32" y1="39.37" x2="18.985" y2="38.035" width="1.016" layer="1"/>
+<via x="11.43" y="22.86" extent="1-16" drill="0.35"/>
+<wire x1="11.43" y1="22.86" x2="11.176" y2="23.114" width="0.1524" layer="16"/>
+<wire x1="11.176" y1="23.114" x2="8.89" y2="23.114" width="0.1524" layer="16"/>
 <wire x1="19.892" y1="28.15" x2="21.38" y2="29.638" width="0" layer="19" extent="1-1"/>
-<wire x1="17.78" y1="25.42" x2="17.78" y2="27.92" width="0" layer="19" extent="1-1"/>
 </signal>
 <signal name="GND">

Commit message: eagle
Routing:
- net +3V3: track 162.8 -> 171.4 mm, vias 4 -> 6
Changed lines of the file:
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@@
 <wire x1="11.43" y1="22.86" x2="11.176" y2="23.114" width="0.1524" layer="16"/>
 <wire x1="11.176" y1="23.114" x2="8.89" y2="23.114" width="0.1524" layer="16"/>
-<wire x1="19.892" y1="28.15" x2="21.38" y2="29.638" width="0" layer="19" extent="1-1"/>
+<via x="13.97" y="30.48" extent="1-16" drill="0.35"/>
+<via x="16.51" y="33.02" extent="1-16" drill="0.35"/>
+<wire x1="16.51" y1="33.02" x2="18.92" y2="33.02" width="0.1524" layer="1"/>
+<wire x1="13.97" y1="30.48" x2="13.97" y2="27.94" width="0.1524" layer="1"/>
+<wire x1="13.97" y1="27.94" x2="13.95" y2="27.92" width="0.1524" layer="1"/>
+<wire x1="13.97" y1="30.48" x2="16.51" y2="33.02" width="0.1524" layer="16"/>
 </signal>
 <signal name="GND">
