File: Sensor_light_system/Eagle/schema Light_system.sch (EAGLE design)
At the start: 23 parts, among them IC1 STM32F030C8T6TR, J1 12_WAY_CON

Commit message: sensor bijgewerkt
Parts:
- U$1: value MODULARCONNECTOR -> I2C_out
- U$2: value MODULARCONNECTOR -> I2C_in
- U$3: value MODULARCONNECTOR -> Program
Connections:
- removed net N$8: IC1.PB2, R3.2
- removed net N$9: IC1.PB0, R1.2
- new net N$3: IC1.PB2, R1.2
- new net N$7: IC1.PB0, R3.2
Changed lines of the file:
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@@
 <part name="C6" library="resistor" deviceset="C-EU" device="C1206" value="100nF"/>
 <part name="GND6" library="supply1" deviceset="GND" device=""/>
-<part name="U$1" library="Main_lib" deviceset="MODULARCONNECTOR" device=""/>
-<part name="U$2" library="Main_lib" deviceset="MODULARCONNECTOR" device=""/>
-<part name="U$3" library="Main_lib" deviceset="MODULARCONNECTOR" device=""/>
+<part name="U$1" library="Main_lib" deviceset="MODULARCONNECTOR" device="" value="I2C_out"/>
+<part name="U$2" library="Main_lib" deviceset="MODULARCONNECTOR" device="" value="I2C_in"/>
+<part name="U$3" library="Main_lib" deviceset="MODULARCONNECTOR" device="" value="Program"/>
 <part name="+3V7" library="supply1" deviceset="+3V3" device=""/>
 <part name="GND7" library="supply1" deviceset="GND" device=""/>
@@
 </segment>
 </net>
+<net name="N$3" class="0">
+<segment>
+<pinref part="R1" gate="G$1" pin="2"/>
+<wire x1="127" y1="63.5" x2="127" y2="68.58" width="0.1524" layer="91"/>
+<wire x1="127" y1="68.58" x2="132.08" y2="68.58" width="0.1524" layer="91"/>
+<pinref part="IC1" gate="G$1" pin="PB2"/>
+<wire x1="132.08" y1="68.58" x2="132.08" y2="71.12" width="0.1524" layer="91"/>
+</segment>
+</net>
+<net name="N$6" class="0">
+<segment>
+<pinref part="IC1" gate="G$1" pin="PB1"/>
+<pinref part="R2" gate="G$1" pin="2"/>
+<wire x1="129.54" y1="71.12" x2="129.54" y2="63.5" width="0.1524" layer="91"/>
+</segment>
+</net>
 <net name="N$7" class="0">
 <segment>
-<pinref part="IC1" gate="G$1" pin="PB1"/>
-<wire x1="129.54" y1="71.12" x2="129.54" y2="63.5" width="0.1524" layer="91"/>
-<pinref part="R2" gate="G$1" pin="2"/>
-</segment>
-</net>
-<net name="N$8" class="0">
-<segment>
-<pinref part="IC1" gate="G$1" pin="PB2"/>
-<wire x1="132.08" y1="71.12" x2="132.08" y2="63.5" width="0.1524" layer="91"/>
+<pinref part="IC1" gate="G$1" pin="PB0"/>
+<wire x1="127" y1="71.12" x2="132.08" y2="66.04" width="0.1524" layer="91"/>
 <pinref part="R3" gate="G$1" pin="2"/>
-</segment>
-</net>
-<net name="N$9" class="0">
-<segment>
-<pinref part="IC1" gate="G$1" pin="PB0"/>
-<pinref part="R1" gate="G$1" pin="2"/>
-<wire x1="127" y1="63.5" x2="127" y2="71.12" width="0.1524" layer="91"/>
-</segment>
-</net>
+<wire x1="132.08" y1="66.04" x2="132.08" y2="63.5" width="0.1524" layer="91"/>
+</segment>
+</net>
