File: Lampen_Light_System/LAMPEN/Lampen.brd (EAGLE design)
At the start: 127 x 49.9 mm, 35 parts, among them T1 BT136, T2 BT136, T3 BT136, T4 BT136, T5 BT136, X1 Lamp0, X2 230VAC, X3 Lamp4, X4 Lamp1, X5 Lamp2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

Commit message: gerbers r2order
Parts:
- moved U$3 27.0 mm to (96.5, 25.1)
- moved U$1 22.0 mm to (80.9, 30.8)
- moved R3 19.0 mm to (49.6, 35.6)
- moved R6 16.9 mm to (72.4, 3.90), turned to 90 degrees
- moved R12 16.1 mm to (72.8, 17.1), turned to 270 degrees
- moved OK2 16.0 mm to (56.4, 40.9)
- moved R10 15.7 mm to (73.3, 10.9), turned to 90 degrees
- moved R13 12.0 mm to (60.4, 17.8)
- moved R14 11.6 mm to (78.9, 17.1), turned to 270 degrees
- moved R8 10.7 mm to (78.9, 24.1), turned to 270 degrees
- moved R11 10.0 mm to (47.1, 17.8)
- moved R1 8.00 mm to (44.1, 44.5)
- moved R9 7.00 mm to (36.2, 17.8)
- moved B1 6.08 mm to (35.9, 39.6)
- moved OK3 6.00 mm to (67.4, 25.4)
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Routing:
- net GND: track 310.8 -> 250.4 mm, vias 1 -> 0
- net SCL: track 192.6 -> 148.2 mm
- net SDA: track 165.3 -> 146.9 mm, vias 0 -> 1
- net 5V: track 242.2 -> 224.5 mm
- net N$25: track 91.4 -> 74.1 mm
- net 3.3V: track 161.8 -> 177.2 mm, vias 0 -> 2
- net N$6: track 99.3 -> 87.8 mm
- net 230VN: track 124.8 -> 113.8 mm
- net N$7: track 25.7 -> 16.9 mm
- net ARD-D6: track 13.6 -> 5.63 mm
- net 230VL: track 126.6 -> 134.2 mm
- net N$4: track 15.1 -> 7.52 mm
- net ARD-D7: track 9.59 -> 3.52 mm
- net N$36: track 16.8 -> 11.5 mm
- net N$30: track 16.8 -> 11.5 mm
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Other:
- board size 127 x 49.9 mm -> 100 x 49.9 mm
